File: hardware/bitsy-v1.1c/icebreaker-bitsy.kicad_sch (KiCad schematic)
At the start: 99 parts, among them J1 USB_C, P0 0, P1 1, P10 10, P11 11, P12 12, P13 13, P14 14, P15 15, P16 16, P17 17, P18 18, P19 19, P2 2, P20 20, P21 21, P22 22, P23 23, P24 GND, P25 GND, P26 GND, P27 3V3, P28 3V3, P29 VIN, P3 3, P30 CDONE, P31 CRESET, P32 UP, P33 UP, P34 UP, P35 UP, P36 CS, P37 SCK, P38 CIPO, P39 COPI, P4 4, P40 IO3, P41 IO2, P5 5, P6 6, P7 7, P8 8, P9 9, SW1 TACT, U1 USBLC6-2, U2 TLV75533PDRV, U3 TLV73312PDRV, U4 LY68L6400, U5 W25Q128JVxxM, U6 ICE40UP5K-SG48, X1 12MHz

Commit message: Adding JLCPCB
Parts:
- C1, C15, C18: LCSC (none) -> C52923
- C10, C14, C17, C6, C7, C8, C9: LCSC (none) -> C1525
- C12: footprint pkl_dipol:C_0402 -> Capacitor_SMD:C_0402_1005Metric; LCSC (none) -> C1525
- C13, C16: LCSC (none) -> C15195
- C19: LCSC (none) -> C19702
- D1: LCSC (none) -> C2286
- D2: LCSC (none) -> C19171392
- D3: LCSC (none) -> C19171394
- D4: LCSC (none) -> C42421005
- J1: LCSC (none) -> C2765186
- R1: LCSC (none) -> C26083
- R10, R7, R8, R9: LCSC (none) -> C25744
- R11: LCSC (none) -> C25879
- R12, R13: footprint pkl_dipol:R_0402 -> Resistor_SMD:R_0402_1005Metric; LCSC (none) -> C25879
- R14: LCSC (none) -> C25076
- R2, R3: LCSC (none) -> C25905
- R4: LCSC (none) -> C25092
- R5: footprint pkl_dipol:R_0402 -> Resistor_SMD:R_0402_1005Metric; LCSC (none) -> C25092
- R6: LCSC (none) -> C25867
- SW1: footprint pkl_buttons_switches:SW_SPST_3x4x2.5 -> Make your own; LCSC (none) -> C720477
- U1: LCSC (none) -> C7519
- U2: LCSC (none) -> C2861750
- U3: LCSC (none) -> C2863369
- U4: LCSC (none) -> C261881
- U5: LCSC (none) -> C2613930
- X1: LCSC (none) -> C9002

Commit message: PCB changes for JLCPCB parts made.
Parts:
- SW1: footprint Make your own -> SWitch:TS-1088-AR02016
Changed lines of the file:
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@@
 			)
 		)
-		(property "Footprint" "Make your own"
+		(property "Footprint" "SWitch:TS-1088-AR02016"
 			(at 91.44 74.295 0)
 			(effects

Commit message: Fixed footprint of U5, etc.
Parts:
- R9: LCSC C25744 -> C326872
- U5: footprint Package_SON:WSON-8-1EP_6x5mm_P1.27mm_EP3.4x4.3mm -> WSON-Library:WSON-8-1EP_6x5mm_P1.27mm_EP3.4x4.3mm; LCSC C2613930 -> C2441427
Changed lines of the file:
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@@
 			)
 		)
-		(property "Footprint" "Package_SON:WSON-8-1EP_6x5mm_P1.27mm_EP3.4x4.3mm"
+		(property "Footprint" "WSON-Library:WSON-8-1EP_6x5mm_P1.27mm_EP3.4x4.3mm"
 			(at 45.72 177.8 0)
 			(effects
@@
 			)
 		)
-		(property "Datasheet" ""
+		(property "Datasheet" "https://jlcpcb.com/api/file/downloadByFileSystemAccessId/8588918790058467328"
 			(at 45.72 177.8 0)
 			(effects
@@
 			)
 		)
-		(property "LCSC" "C2613930"
+		(property "LCSC" "C2441427"
 			(at 45.72 177.8 0)
 			(effects
@@
 			)
 		)
-		(property "LCSC" "C25744"
+		(property "LCSC" "C326872"
 			(at 73.66 142.24 90)
 			(effects
@@
 			)
 		)
-		(property "LCSC" "C25744"
+		(property "LCSC" "C326872"
 			(at 76.2 142.24 90)
 			(effects
@@
 			)
 		)
-		(property "LCSC" "C25744"
+		(property "LCSC" "C326872"
 			(at 276.86 114.3 90)
 			(effects
@@
 			)
 		)
-		(property "LCSC" "C25744"
+		(property "LCSC" "C326872"
 			(at 71.12 142.24 90)
 			(effects
